Commit message: fds

File: body.urdf (robot description, URDF)
Before this commit: robot robot, 3 links, 2 joints
Links:
- added link BackLowerLeg, mass 1; collision box size=0.2 0.2 1; visual box size=0.2 0.2 1
- added link FrontLowerLeg, mass 1; collision box size=0.2 0.2 1; visual box size=0.2 0.2 1
- added link LeftLeg, mass 1; collision box size=1 0.2 0.2; visual box size=1 0.2 0.2
- added link LeftLowerLeg, mass 1; collision box size=0.2 0.2 1; visual box size=0.2 0.2 1
- added link RightLeg, mass 1; collision box size=1 0.2 0.2; visual box size=1 0.2 0.2
- added link RightLowerLeg, mass 1; collision box size=0.2 0.2 1; visual box size=0.2 0.2 1
- link BackLeg: geometry collision box size=0.2 1 0.2; visual box size=0.2 1 0.2
- link FrontLeg: geometry collision box size=0.2 1 0.2; visual box size=0.2 1 0.2
Joints:
- added joint BackLeg_BackLowerLeg: type revolute, parent BackLeg, child BackLowerLeg, origin xyz=0 -1 0 rpy=0 0 0, axis 1 0 0, limit lower=-3.14159 upper=3.14159 effort=0.0 velocity=0.0
- added joint FrontLeg_FrontLowerLeg: type revolute, parent FrontLeg, child FrontLowerLeg, origin xyz=0 1 0 rpy=0 0 0, axis 1 0 0, limit lower=-3.14159 upper=3.14159 effort=0.0 velocity=0.0
- added joint LeftLeg_LeftLowerLeg: type revolute, parent LeftLeg, child LeftLowerLeg, origin xyz=-1 0 0 rpy=0 0 0, axis 0 1 0, limit lower=-3.14159 upper=3.14159 effort=0.0 velocity=0.0
- added joint RightLeg_RightLowerLeg: type revolute, parent RightLeg, child RightLowerLeg, origin xyz=1 0 0 rpy=0 0 0, axis 0 1 0, limit lower=-3.14159 upper=3.14159 effort=0.0 velocity=0.0
- added joint Torso_LeftLeg: type revolute, parent Torso, child LeftLeg, origin xyz=-0.5 0 1.0 rpy=0 0 0, axis 0 1 0, limit lower=-3.14159 upper=3.14159 effort=0.0 velocity=0.0
- added joint Torso_RightLeg: type revolute, parent Torso, child RightLeg, origin xyz=0.5 0 1.0 rpy=0 0 0, axis 0 1 0, limit lower=-3.14159 upper=3.14159 effort=0.0 velocity=0.0
- joint Torso_BackLeg: axis 0 1 0 -> 1 0 0; origin xyz=1 0 1.0 rpy=0 0 0 -> xyz=0 -0.5 1.0 rpy=0 0 0
- joint Torso_FrontLeg: axis 0 1 0 -> 1 0 0; origin xyz=2 0 1.0 rpy=0 0 0 -> xyz=0 0.5 1.0 rpy=0 0 0

Commit message: hexapod

File: body.urdf (robot description, URDF)
Before this commit: robot robot, 9 links, 8 joints
Links:
- added link LLLeg, mass 1; collision box size=0.2 0.2 1; visual box size=0.2 0.2 1
- added link LLeg, mass 1; collision box size=1 0.2 0.2; visual box size=1 0.2 0.2
- added link RLeg, mass 1; collision box size=1 0.2 0.2; visual box size=1 0.2 0.2
- added link RRLeg, mass 1; collision box size=0.2 0.2 1; visual box size=0.2 0.2 1
Joints:
- added joint LLeg_LLLeg: type revolute, parent LLeg, child LLLeg, origin xyz=-1 0 0 rpy=0 0 0, axis 0 1 0, limit lower=-3.14159 upper=3.14159 effort=0.0 velocity=0.0
- added joint RLeg_RRLeg: type revolute, parent RLeg, child RRLeg, origin xyz=1 0 0 rpy=0 0 0, axis 0 1 0, limit lower=-3.14159 upper=3.14159 effort=0.0 velocity=0.0
- added joint Torso_LLeg: type revolute, parent Torso, child LLeg, origin xyz=-0.5 0.5 1.0 rpy=0 0 0, axis 0 1 0, limit lower=-3.14159 upper=3.14159 effort=0.0 velocity=0.0
- added joint Torso_RLeg: type revolute, parent Torso, child RLeg, origin xyz=0.5 0.5 1.0 rpy=0 0 0, axis 0 1 0, limit lower=-3.14159 upper=3.14159 effort=0.0 velocity=0.0

Commit message: hexapod jump

File: body.urdf (robot description, URDF)
Before this commit: robot robot, 13 links, 12 joints
Joints:
- joint Torso_LLeg: origin xyz=-0.5 0.5 1.0 rpy=0 0 0 -> xyz=-0.5 0.2 1.0 rpy=0 0 0
- joint Torso_LeftLeg: origin xyz=-0.5 0 1.0 rpy=0 0 0 -> xyz=-0.5 -0.2 1.0 rpy=0 0 0
- joint Torso_RLeg: origin xyz=0.5 0.5 1.0 rpy=0 0 0 -> xyz=0.5 0.2 1.0 rpy=0 0 0
- joint Torso_RightLeg: origin xyz=0.5 0 1.0 rpy=0 0 0 -> xyz=0.5 -0.2 1.0 rpy=0 0 0

Commit message: snake done

File: body.urdf (robot description, URDF)
Before this commit: robot robot, 13 links, 12 joints
Links:
- removed link BackLeg
- removed link BackLowerLeg
- removed link FrontLeg
- removed link FrontLowerLeg
- removed link LLLeg
- removed link LLeg
- removed link LeftLeg
- removed link LeftLowerLeg
- removed link RLeg
- removed link RRLeg
- removed link RightLeg
- removed link RightLowerLeg
- removed link Torso
- added link 0, mass 1; collision box size=0.8801447603657874 0.7717467477737991 0.30795962220962725; visual box size=0.8801447603657874 0.7717467477737991 0.30795962220962725
- added link 1, mass 1; collision box size=0.7346801064328097 1.1029631443283445 0.78265498358222; visual box size=0.7346801064328097 1.1029631443283445 0.78265498358222
- added link 2, mass 1; collision box size=0.9944124190785801 1.1836747852173577 0.723542009985554; visual box size=0.9944124190785801 1.1836747852173577 0.723542009985554
- added link 3, mass 1; collision box size=0.9761360650199129 0.8264119967875764 0.8347351230273897; visual box size=0.9761360650199129 0.8264119967875764 0.8347351230273897
- added link 4, mass 1; collision box size=1.0565063009827247 1.2106845735693055 0.2761829228865741; visual box size=1.0565063009827247 1.2106845735693055 0.2761829228865741
- added link 5, mass 1; collision box size=0.4795319004287768 0.8561941554088136 1.0932675707985477; visual box size=0.4795319004287768 0.8561941554088136 1.0932675707985477
- added link 6, mass 1; collision box size=0.9135501305245811 0.507731457026881 0.5822205524043724; visual box size=0.9135501305245811 0.507731457026881 0.5822205524043724
- added link 7, mass 1; collision box size=0.6841549876004006 1.1029530517021517 0.7970969899854914; visual box size=0.6841549876004006 1.1029530517021517 0.7970969899854914
Joints:
- removed joint BackLeg_BackLowerLeg
- removed joint FrontLeg_FrontLowerLeg
- removed joint LLeg_LLLeg
- removed joint LeftLeg_LeftLowerLeg
- removed joint RLeg_RRLeg
- removed joint RightLeg_RightLowerLeg
- removed joint Torso_BackLeg
- removed joint Torso_FrontLeg
- removed joint Torso_LLeg
- removed joint Torso_LeftLeg
- removed joint Torso_RLeg
- removed joint Torso_RightLeg
- added joint 0_1: type revolute, parent 0, child 1, origin xyz=0 0.7717467477737991 0.15397981110481362 rpy=0 0 0, axis 0 0 1, limit lower=-3.14159 upper=3.14159 effort=0.0 velocity=0.0
- added joint 1_2: type revolute, parent 1, child 2, origin xyz=0 1.1029631443283445 0.23734768068629636 rpy=0 0 0, axis 0 0 1, limit lower=-3.14159 upper=3.14159 effort=0.0 velocity=0.0
- added joint 2_3: type revolute, parent 2, child 3, origin xyz=0 1.1836747852173577 -0.029556486798333004 rpy=0 0 0, axis 0 0 1, limit lower=-3.14159 upper=3.14159 effort=0.0 velocity=0.0
- added joint 3_4: type revolute, parent 3, child 4, origin xyz=0 0.8264119967875764 0.055596556520917884 rpy=0 0 0, axis 0 0 1, limit lower=-3.14159 upper=3.14159 effort=0.0 velocity=0.0
- added joint 4_5: type revolute, parent 4, child 5, origin xyz=0 1.2106845735693055 -0.2792761000704078 rpy=0 0 0, axis 0 0 1, limit lower=-3.14159 upper=3.14159 effort=0.0 velocity=0.0
- added joint 5_6: type revolute, parent 5, child 6, origin xyz=0 0.8561941554088136 0.40854232395598683 rpy=0 0 0, axis 0 0 1, limit lower=-3.14159 upper=3.14159 effort=0.0 velocity=0.0
- added joint 6_7: type revolute, parent 6, child 7, origin xyz=0 0.507731457026881 -0.25552350919708766 rpy=0 0 0, axis 0 0 1, limit lower=-3.14159 upper=3.14159 effort=0.0 velocity=0.0
